File: PCB/projet_hmae.kicad_pcb (KiCad board)
At the start: 2 copper layers, 87.2 x 63.8 mm, 21 parts, among them J1 DM3CS-SF, J2 Conn_01x11_Female, J4 Conn_01x05_Female, U2 ESP32-WROOM-32, U3 LM317L_SOT-89

Commit message: YEP
Parts:
- added R4: 100kOhms, Resistor_SMD:R_1206_3216Metric_Pad1.30x1.75mm_HandSolder, F.Cu at (128.7, 34.8)
- renumbered LM386 to U1, NE555 to U4
Routing:
- net Net-(PlantInput1-Pad1): track 18.5 -> 27.9 mm
- net +3V3: track 153.5 -> 158.3 mm
Changed lines of the file:
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@@
   (net 24 "ESP32_RX")
   (net 25 "ESP32_TX")
-  (net 26 "Net-(U2-Pad25)")
+  (net 26 "Net-(BOOT1-Pad1)")
   (net 27 "unconnected-(PlantInput1-Pad3)")
   (net 28 "Net-(R2-Pad2)")
@@
   (net 54 "Net-(J2-Pad9)")
   (net 55 "Net-(PlantInput1-Pad1)")
-  (net 56 "Net-(U2-Pad3)")
+  (net 56 "Net-(RST1-Pad2)")
   (net 57 "unconnected-(Power1-Pad3)")
   (footprint "Package_TO_SOT_SMD:SOT-89-3" (layer "F.Cu")
@@
     (fp_circle (center 0 0) (end 1.7 0) (layer "F.Fab") (width 0.1) (fill none))
     (pad "1" smd rect (at -2.88 -2) (size 2.75 1) (layers "F.Cu" "F.Paste" "F.Mask")
-      (net 26 "Net-(U2-Pad25)") (pinfunction "1") (pintype "passive"))
+      (net 26 "Net-(BOOT1-Pad1)") (pinfunction "1") (pintype "passive"))
     (pad "1" smd rect (at 2.88 -2) (size 2.75 1) (layers "F.Cu" "F.Paste" "F.Mask")
-      (net 26 "Net-(U2-Pad25)") (pinfunction "1") (pintype "passive"))
+      (net 26 "Net-(BOOT1-Pad1)") (pinfunction "1") (pintype "passive"))
     (pad "2" smd rect (at -2.88 2) (size 2.75 1) (layers "F.Cu" "F.Paste" "F.Mask")
       (net 2 "GND") (pinfunction "2") (pintype "passive"))
@@
       (net 12 "+3V3") (pinfunction "VDD") (pintype "power_in"))
     (pad "3" smd rect (at -8.5 -5.715 90) (size 2 0.9) (layers "F.Cu" "F.Paste" "F.Mask")
-      (net 56 "Net-(U2-Pad3)") (pinfunction "EN") (pintype "input"))
+      (net 56 "Net-(RST1-Pad2)") (pinfunction "EN") (pintype "input"))
     (pad "4" smd rect (at -8.5 -4.445 90) (size 2 0.9) (layers "F.Cu" "F.Paste" "F.Mask")
       (net 32 "unconnected-(U2-Pad4)") (pinfunction "SENSOR_VP") (pintype "input+no_connect"))
@@
       (net 36 "unconnected-(U2-Pad24)") (pinfunction "IO2") (pintype "bidirectional+no_connect"))
     (pad "25" smd rect (at 8.5 8.255 90) (size 2 0.9) (layers "F.Cu" "F.Paste" "F.Mask")
-      (net 26 "Net-(U2-Pad25)") (pinfunction "IO0") (pintype "bidirectional"))
+      (net 26 "Net-(BOOT1-Pad1)") (pinfunction "IO0") (pintype "bidirectional"))
     (pad "26" smd rect (at 8.5 6.985 90) (size 2 0.9) (layers "F.Cu" "F.Paste" "F.Mask")
       (net 38 "555Output") (pinfunction "IO4") (pintype "bidirectional"))
@@
       (scale (xyz 1 1 1))
       (rotate (xyz 0 -180 0))
+    )
+  )
+  (footprint "Resistor_SMD:R_1206_3216Metric_Pad1.30x1.75mm_HandSolder" (layer "F.Cu")
+    (at 128.65 34.8)
+    (descr "Resistor SMD 1206 (3216 Metric), square (rectangular) end terminal, IPC_7351 nominal with elongated pad for handsoldering. (Body size source: IPC-SM-782 page 72, https://www.pcb-3d.com/wordpress/wp-content/uploads/ipc-sm-782a_amendment_1_and_2.pdf), generated with kicad-footprint-generator")
+    (tags "resistor handsolder")
+    (property "Sheetfile" "projet_hmae.kicad_sch")
+    (property "Sheetname" "")
+    (attr smd)
+    (fp_text reference "R4" (at 0 -1.82) (layer "F.SilkS")
+      (effects (font (size 1 1) (thickness 0.15)))
+    )
+    (fp_text value "100kOhms" (at 0 1.82) (layer "F.Fab")
+      (effects (font (size 1 1) (thickness 0.15)))
+    )
+    (fp_text user "${REFERENCE}" (at 0 0) (layer "F.Fab")
+      (effects (font (size 0.8 0.8) (thickness 0.12)))
+    )
+    (fp_line (start -0.727064 -0.91) (end 0.727064 -0.91) (layer "F.SilkS") (width 0.12))
+    (fp_line (start -0.727064 0.91) (end 0.727064 0.91) (layer "F.SilkS") (width 0.12))
+    (fp_line (start -2.45 -1.12) (end 2.45 -1.12) (layer "F.CrtYd") (width 0.05))
+    (fp_line (start 2.45 1.12) (end -2.45 1.12) (layer "F.CrtYd") (width 0.05))
+    (fp_line (start -2.45 1.12) (end -2.45 -1.12) (layer "F.CrtYd") (width 0.05))
+    (fp_line (start 2.45 -1.12) (end 2.45 1.12) (layer "F.CrtYd") (width 0.05))
+    (fp_line (start 1.6 0.8) (end -1.6 0.8) (layer "F.Fab") (width 0.1))
+    (fp_line (start -1.6 0.8) (end -1.6 -0.8) (layer "F.Fab") (width 0.1))
+    (fp_line (start -1.6 -0.8) (end 1.6 -0.8) (layer "F.Fab") (width 0.1))
+    (fp_line (start 1.6 -0.8) (end 1.6 0.8) (layer "F.Fab") (width 0.1))
+    (pad "1" smd roundrect (at -1.55 0) (size 1.3 1.75) (layers "F.Cu" "F.Paste" "F.Mask") (roundrect_rratio 0.192308)
+      (net 12 "+3V3") (pintype "passive"))
+    (pad "2" smd roundrect (at 1.55 0) (size 1.3 1.75) (layers "F.Cu" "F.Paste" "F.Mask") (roundrect_rratio 0.192308)
+      (net 55 "Net-(PlantInput1-Pad1)") (pintype "passive"))
+    (model "${KICAD6_3DMODEL_DIR}/Resistor_SMD.3dshapes/R_1206_3216Metric.wrl"
+      (offset (xyz 0 0 0))
+      (scale (xyz 1 1 1))
+      (rotate (xyz 0 0 0))
     )
   )
@@
     (property "Sheetname" "")
     (attr through_hole)
-    (fp_text reference "LM386" (at 0 -6.2 90) (layer "F.SilkS")
+    (fp_text reference "U1" (at 0 -6.2 90) (layer "F.SilkS")
       (effects (font (size 1 1) (thickness 0.15)))
     )
@@
       (net 2 "GND") (pinfunction "1") (pintype "passive"))
     (pad "2" smd rect (at -2.88 2 180) (size 2.75 1) (layers "F.Cu" "F.Paste" "F.Mask")
-      (net 56 "Net-(U2-Pad3)") (pinfunction "2") (pintype "passive"))
+      (net 56 "Net-(RST1-Pad2)") (pinfunction "2") (pintype "passive"))
     (pad "2" smd rect (at 2.88 2 180) (size 2.75 1) (layers "F.Cu" "F.Paste" "F.Mask")
-      (net 56 "Net-(U2-Pad3)") (pinfunction "2") (pintype "passive"))
+      (net 56 "Net-(RST1-Pad2)") (pinfunction "2") (pintype "passive"))
     (model "${KICAD6_3DMODEL_DIR}/Button_Switch_SMD.3dshapes/SW_SPST_EVQP0.wrl"
       (offset (xyz 0 0 0))
@@
     (property "Sheetname" "")
     (attr through_hole)
-    (fp_text reference "NE555" (at 3.81 -2.33) (layer "F.SilkS")
+    (fp_text reference "U4" (at 3.81 -2.33) (layer "F.SilkS")
       (effects (font (size 1 1) (thickness 0.15)))
     )
@@
   (segment (start 95 52.2375) (end 95 58.7) (width 0.25) (layer "F.Cu") (net 12))
   (segment (start 115.4 44.22) (end 111.98 44.22) (width 0.25) (layer "F.Cu") (net 12))
+  (segment (start 123.02 36.6) (end 125.3 36.6) (width 0.25) (layer "F.Cu") (net 12))
   (segment (start 64.415 69.7) (end 64.415 73.255) (width 0.25) (layer "F.Cu") (net 12))
   (segment (start 64.415 73.255) (end 66.96 75.8) (width 0.25) (layer "F.Cu") (net 12))
@@
   (segment (start 111.98 44.22) (end 106.075489 50.124511) (width 0.25) (layer "F.Cu") (net 12))
   (segment (start 66.885978 66.4) (end 64.415 68.870978) (width 0.25) (layer "F.Cu") (net 12))
+  (segment (start 125.3 36.6) (end 127.1 34.8) (width 0.25) (layer "F.Cu") (net 12))
   (segment (start 64.415 68.870978) (end 64.415 69.7) (width 0.25) (layer "F.Cu") (net 12))
   (segment (start 138.2 56) (end 138.2 58.425) (width 0.25) (layer "F.Cu") (net 12))
@@
   (segment (start 69.495 75.795) (end 69.5 75.8) (width 0.25) (layer "F.Cu") (net 54))
   (segment (start 69.495 69.7) (end 69.495 75.795) (width 0.25) (layer "F.Cu") (net 54))
+  (segment (start 131.489 33.511) (end 139.15 33.511) (width 0.25) (layer "F.Cu") (net 55))
+  (segment (start 130.2 34.8) (end 131.489 33.511) (width 0.25) (layer "F.Cu") (net 55))
   (segment (start 123.02 39.14) (end 133.521 39.14) (width 0.25) (layer "F.Cu") (net 55))
   (segment (start 133.521 39.14) (end 139.15 33.511) (width 0.25) (layer "F.Cu") (net 55))
