File: PCB/projet_hmae.kicad_sch (KiCad schematic)
At the start: 21 parts, among them J1 DM3CS-SF, J2 Conn_01x11_Female, J4 Conn_01x05_Female, U1 LM386, U2 ESP32-WROOM-32, U3 LM317L_SOT-89, U4 NE555P

Commit message: YEP
Parts:
- added R4: 100kOhms, Resistor_SMD:R_1206_3216Metric_Pad1.30x1.75mm_HandSolder, symbol Device:R
Connections:
- net +3V3: now also R4.1
- net at PlantInput1.1, U4.7 (DIS): now also R4.2
Changed lines of the file:
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@@
   (junction (at 353.06 220.98) (diameter 0) (color 0 0 0 0)
   )
+  (junction (at 337.82 191.77) (diameter 0) (color 0 0 0 0)
+  )
   (junction (at 367.03 45.72) (diameter 0) (color 0 0 0 0)
   )
@@
   )
   (junction (at 353.06 213.36) (diameter 0) (color 0 0 0 0)
+  )
+  (junction (at 369.57 208.28) (diameter 0) (color 0 0 0 0)
   )
   (junction (at 337.82 27.94) (diameter 0) (color 0 0 0 0)
@@
     (stroke (width 0) (type default) (color 0 0 0 0))
   )
-  (wire (pts (xy 337.82 190.5) (xy 337.82 198.12))
+  (wire (pts (xy 337.82 190.5) (xy 337.82 191.77))
     (stroke (width 0) (type default) (color 0 0 0 0))
   )
@@
     (stroke (width 0) (type default) (color 0 0 0 0))
   )
+  (wire (pts (xy 337.82 191.77) (xy 369.57 191.77))
+    (stroke (width 0) (type default) (color 0 0 0 0))
+  )
   (wire (pts (xy 34.29 162.56) (xy 48.26 162.56))
     (stroke (width 0) (type default) (color 0 0 0 0))
@@
     (stroke (width 0) (type default) (color 0 0 0 0))
   )
+  (wire (pts (xy 369.57 191.77) (xy 369.57 196.85))
+    (stroke (width 0) (type default) (color 0 0 0 0))
+  )
   (wire (pts (xy 337.82 218.44) (xy 337.82 220.98))
     (stroke (width 0) (type default) (color 0 0 0 0))
@@
     (stroke (width 0) (type default) (color 0 0 0 0))
   )
+  (wire (pts (xy 337.82 191.77) (xy 337.82 198.12))
+    (stroke (width 0) (type default) (color 0 0 0 0))
+  )
   (wire (pts (xy 158.75 93.98) (xy 158.75 96.52))
     (stroke (width 0) (type default) (color 0 0 0 0))
@@
     (stroke (width 0) (type default) (color 0 0 0 0))
   )
+  (wire (pts (xy 369.57 208.28) (xy 374.65 208.28))
+    (stroke (width 0) (type default) (color 0 0 0 0))
+  )
+  (wire (pts (xy 369.57 204.47) (xy 369.57 208.28))
+    (stroke (width 0) (type default) (color 0 0 0 0))
+  )
   (wire (pts (xy 316.23 203.2) (xy 316.23 194.31))
     (stroke (width 0) (type default) (color 0 0 0 0))
@@
     (stroke (width 0) (type default) (color 0 0 0 0))
   )
-  (wire (pts (xy 350.52 208.28) (xy 374.65 208.28))
+  (wire (pts (xy 350.52 208.28) (xy 369.57 208.28))
     (stroke (width 0) (type default) (color 0 0 0 0))
   )
@@
     (pin "7")
   )
+  (symbol (lib_id "Device:R") (at 369.57 200.66 0) (unit 1)
+    (in_bom yes) (on_board yes) (fields_autoplaced)
+    (property "Reference" "R4" (id 0) (at 372.11 199.3899 0)
+      (effects (font (size 1.27 1.27)) (justify left))
+    )
+    (property "Value" "100kOhms" (id 1) (at 372.11 201.9299 0)
+      (effects (font (size 1.27 1.27)) (justify left))
+    )
+    (property "Footprint" "Resistor_SMD:R_1206_3216Metric_Pad1.30x1.75mm_HandSolder" (id 2) (at 367.792 200.66 90)
+      (effects (font (size 1.27 1.27)) hide)
+    )
+    (property "Datasheet" "~" (id 3) (at 369.57 200.66 0)
+      (effects (font (size 1.27 1.27)) hide)
+    )
+    (pin "1")
+    (pin "2")
+  )
   (symbol (lib_id "Device:R_Potentiometer") (at 45.72 34.29 0) (unit 1)
     (in_bom yes) (on_board yes) (fields_autoplaced)
@@
       (reference "R3") (unit 1) (value "1639Ohm") (footprint "Resistor_SMD:R_1206_3216Metric_Pad1.30x1.75mm_HandSolder")
     )
+    (path "/c84e14d3-e4ed-44aa-a72a-e3cd27cfffa7"
+      (reference "R4") (unit 1) (value "100kOhms") (footprint "Resistor_SMD:R_1206_3216Metric_Pad1.30x1.75mm_HandSolder")
+    )
     (path "/1a9e2b11-80b9-435f-a9bf-a5b45e4a1043"
